Commit message: Revert "Added Dual UR5 Husky"

File: husky_description/urdf/decorations.urdf.xacro (robot description, xacro)
@@ -37,20 +37,18 @@
       <child link="top_chassis_link" />
     </joint>
-    <xacro:if value="$(optenv HUSKY_USER_RAILS true)">
-	    <!-- Spawn user rails -->
-	    <link name="user_rail_link">
-	      <visual>
-		<geometry>
-		  <mesh filename="package://husky_description/meshes/user_rail.dae" />
-		</geometry>
-	      </visual>
-	    </link>
-	    <!-- Attach user rails to base link -->
-	    <joint name="user_rail" type="fixed">
-	      <origin xyz="0.272 0 0.245" rpy="0 0 0" />
-	      <parent link="base_link" />
-	      <child link="user_rail_link" />
-	    </joint>
-    </xacro:if>
+    <!-- Spawn user rails -->
+    <link name="user_rail_link">
+      <visual>
+        <geometry>
+          <mesh filename="package://husky_description/meshes/user_rail.dae" />
+        </geometry>
+      </visual>
+    </link>
+    <!-- Attach user rails to base link -->
+    <joint name="user_rail" type="fixed">
+      <origin xyz="0.272 0 0.245" rpy="0 0 0" />
+      <parent link="base_link" />
+      <child link="user_rail_link" />
+    </joint>
     <!-- Spawn front bumper link -->
     <link name="front_bumper_link">
@@ -81,32 +79,4 @@
       <child link="rear_bumper_link" />
     </joint>
-    <xacro:if value="$(optenv DUAL_ARM_BULKHEAD false)">
-        <!-- Spawn the bulkhead -->
-        <link name="dual_arm_bulkhead_link">
-        <visual>
-          <origin xyz="0 0 0" rpy="0 0 0" />
-          <geometry>
-            <mesh filename="package://husky_description/meshes/dual_arm_bulkhead.dae" />
-          </geometry>
-        </visual>
-        <collision>
-          <origin xyz="0 0 0" rpy="0 0 0"/>
-           <geometry>
-            <mesh filename="package://husky_description/meshes/dual_arm_bulkhead.dae" />
-          </geometry>
-        </collision>
-          <inertial>
-            <mass value="9.832"/>
-            <origin xyz="0 0 0" />
-            <inertia ixx="0.177184" ixy="-0.0045887" ixz="0.003812" iyy="0.752238" iyz="0.004194" izz="0.1376" />
-          </inertial>
-        </link>
-      <!-- Attach bulkhead -->
-      <joint name="dual_arm_bulkhead_joint" type="fixed">
-        <parent link="base_link" />
-        <child link="dual_arm_bulkhead_link"/>
-        <origin xyz="0 0 0.225" rpy="0 0 0"/>
-      </joint>
-    </xacro:if>
     <xacro:if value="$(optenv HUSKY_TOP_PLATE_ENABLED true)">
       <!-- Spawn the top plate -->

File: husky_description/urdf/description.xacro (robot description, xacro)
@@ -22,10 +22,8 @@
 -->
 <robot name="husky" xmlns:xacro="http://ros.org/wiki/xacro">
-  <xacro:arg name="dual_ur5_enabled" default="$(optenv HUSKY_DUAL_UR5_ENABLED false)" />
   <xacro:arg name="laser_enabled" default="false" />
   <xacro:arg name="ur5_enabled" default="false" />
   <xacro:arg name="kinect_enabled" default="false" />
-  <xacro:arg name="robotiq_grippers_enabled" default="$(optenv ROBOTIQ_GRIPPERS_ENABLED false)" />
-  <xacro:include filename="$(find husky_description)/urdf/dual_arm_husky.urdf.xacro" />
+  <xacro:include filename="$(find husky_description)/urdf/husky.urdf.xacro" />
   <xacro:husky_robot />
 </robot>

File: husky_description/urdf/husky.urdf.xacro (robot description, xacro)
@@ -29,8 +29,4 @@
   <xacro:include filename="$(find husky_description)/urdf/accessories/sensor_arch.urdf.xacro"/>
   <xacro:include filename="$(find ur_description)/urdf/ur5.urdf.xacro" />
-  <xacro:include filename="$(find robotiq_s_model_visualization)/cfg/robotiq_hand_macro.urdf.xacro"/>
-  <xacro:include filename="$(find robotiq_force_torque_sensor)/urdf/robotiq_fts300.urdf.xacro"/>
-  <xacro:include filename="$(find flir_ptu_description)/urdf/d46.urdf.xacro"/>
-  <xacro:include filename="$(find pointgrey_camera_description)/urdf/pointgrey_bumblebee2.urdf.xacro"/>
   <property name="M_PI" value="3.14159"/>
   <!-- Base Size -->
@@ -74,17 +70,9 @@
       <child link="base_footprint" />
     </joint>
-<<<<<<< HEAD
     <!-- Interial link stores the robot's inertial information -->
     <link name="inertial_link">
       <inertial>
-        <mass value="46.034"/>
-        <origin xyz="-0.00065 -0.085 0.062" />
-=======
-    <!-- Interial link stores the robot's inertial information
-    <link name="inertial_link">
-      <inertial>
-        <mass value="" />
+        <mass value="33.455" />
         <origin xyz="-0.08748 -0.00085 0.09947" />
->>>>>>> 685a629... Shits broken
         <inertia ixx="0.6022" ixy="-0.02364" ixz="-0.1197" iyy="1.7386" iyz="-0.001544" izz="2.0296" />
       </inertial>
@@ -94,9 +82,5 @@
       <parent link="base_link" />
       <child link="inertial_link" />
-<<<<<<< HEAD
     </joint>
-=======
-    </joint> -->
->>>>>>> 685a629... Shits broken
     <!-- IMU Link is the standard mounting position for the UM6 IMU.-->
     <!-- Can be modified with environment variables in /etc/ros/setup.bash -->
@@ -123,59 +107,4 @@
     </xacro:husky_wheel>
     <xacro:husky_decorate />
-    <xacro:if value="$(optenv FLIR_PTU_ENABLED false)">
-          <xacro:ptu_d46 name="husky_ptu"/>
-          <!-- Connect PTU to Husky bulkhead -->
-          <joint name="husky_ptu_joint" type="fixed">
-             <origin xyz="0.365 0 0.20" rpy="0 0 0"/>
-             <parent link="dual_arm_bulkhead_link" />
-             <child link="husky_ptu_base_link" />
-         </joint>
-    </xacro:if>
-    <xacro:if value="$(optenv HUSKY_DUAL_UR5_ENABLED false)">
-        <xacro:ur5_robot prefix="l_ur5_arm_" joint_limited="true"/>
-        <xacro:ur5_robot prefix="r_ur5_arm_" joint_limited="true"/>
-        <!-- Add laser specifically for this mode -->
-        <sick_lms1xx frame="base_laser" topic="scan" />
-        <!-- This offset is from the base of the bracket to the LIDAR's focal point. -->
-        <joint name="base_laser_joint" type="fixed">
-           <origin xyz="0.465 0 -0.085" rpy="${M_PI} 0 0" />
-           <parent link="dual_arm_bulkhead_link" />
-           <child link="base_laser" />
-        </joint>
-        <!-- Add bumblebee camera -->
-       <BB2-08S2C-38 frame="bumblebee2" name="bumblebee2" />
-        <joint name="bumblebee2_mount_joint" type="fixed">
-           <origin xyz="0 0 0.00" rpy="0 0 0" />
-           <parent link="husky_ptu_mount_link" />
-           <child link="bumblebee2" />
-        </joint>
-        <!-- Add force torque model FT300 -->
-        <xacro:robotiq_fts300 parent="l_ur5_arm_ee_link" prefix="l_robotiq_fts300_">
-           <origin xyz="0 0 0" rpy="0 1.57 0"/>
-        </xacro:robotiq_fts300>
-        <xacro:robotiq_fts300 parent="r_ur5_arm_ee_link" prefix="r_robotiq_fts300_">
-           <origin xyz="0 0 0" rpy="0 1.57 0"/>
-        </xacro:robotiq_fts300>
-        <xacro:if value="$(optenv ROBOTIQ_GRIPPERS_ENABLED false)">
-            <xacro:robotiq_hand prefix="l_" reflect="1" parent="l_robotiq_fts300_fts_toolside">
-                <origin xyz="0 0 0.08" rpy="1.57 0 0"/>
-            </xacro:robotiq_hand>
-            <xacro:robotiq_hand prefix="r_" reflect="1" parent="r_robotiq_fts300_fts_toolside">
-                <origin xyz="0 0 0.08" rpy="1.57 0 0"/>
-            </xacro:robotiq_hand>
-        </xacro:if>
-        <!-- Join left arm to top plate -->
-        <joint name="r_ur5_arm_base" type="fixed">
-            <parent link="dual_arm_bulkhead_link"/>
-            <child link="r_ur5_arm_base_link" />
-            <origin xyz="0.125 -0.15 0.135" rpy="0 0.785 -1.57"/>
-        </joint>
-         <!-- Joint right arm to top plate -->
-        <joint name="l_ur5_arm_base" type="fixed">
-            <parent link="dual_arm_bulkhead_link"/>
-            <child link="l_ur5_arm_base_link" />
-            <origin xyz="0.125 0.15 0.135" rpy="0 -0.785 -1.57"/>
-        </joint>
-    </xacro:if>
     <xacro:if value="$(arg ur5_enabled)">
       <xacro:property name="reflect" value="-1" />
@@ -189,10 +118,10 @@
       </joint>
     </xacro:if>
-    <xacro:if value="$(optenv HUSKY_LASER_ENABLED false)">
+    <xacro:if value="$(arg laser_enabled)">
       <sick_lms1xx_mount prefix="base" topic="scan"/>
       <joint name="laser_mount_joint" type="fixed">
         <origin xyz="$(optenv HUSKY_LMS1XX_XYZ 0.2206 0.0 0.00635)"
                 rpy="$(optenv HUSKY_LMS1XX_RPY 0.0 0.0 0.0)" />
-        <parent link="$(optenv HUSKY_LASER_PARENT_LINK top_plate_link)" />
+        <parent link="top_plate_link" />
         <child link="base_laser_mount" />
       </joint>
